File: extras/clock_10/eagle/clock10.sch (EAGLE design)
At the start: 120 parts, among them IC101 DC-DC-STEP-DOWN-LM2596, IC102 DS3231W, IC103 1117 3V3, IC104 ZOPT2201, IC105 BME280, IC106 74AC245DW, IC107 74AC245DW, IC201 ESP32S2, IC202 ESP12F, IC203 ESP32C3-MODULE13U, IC204 ESP12F, IC301 1117 3V3, IC302 BME280, J101 12V, J102 IN, J104 4P-2.0, J105 4P-2.0, J201 USB_1, J202 COM, J203 COM, J204 COM, J205 COM, J206 USB_2, J207 OUT_2, J208 OUT_1, J209 OUT_3, J301 IN, SW101 PRG, SW102 RST, U101 SI7021, U301 SI7021, X101 +5V, X102 SHT22, X103 AM2320, X301 +5V, X302 DHT22, X303 AM2320

Commit message: add s2
Connections:
- net I33 renamed 1IO33
- net IO16 renamed 1IO16
- net IO17 renamed 1IO17
- net IO18 renamed 1IO18
- net IO21 renamed 1IO21
- net IO26 renamed 1IO26
- net IO38 renamed 1IO38
- net IO42 renamed 1IO42
- removed net IO15: IC201.I15
- new net 1IO15: IC201.I15, J208.8
- net 1IO0: now also J202.6, J208.2
- net 1IO1: now also J208.9
- net 1IO2: now also J208.10; no longer J208.8
- net 1IO35: no longer J202.6, J208.2
- net 1IO45: no longer J208.9
- net 1IO46: no longer J208.10
Changed lines of the file:
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@@
 </segment>
 </net>
-<net name="IO38" class="0">
+<net name="1IO38" class="0">
 <segment>
 <wire x1="40.64" y1="50.8" x2="43.18" y2="50.8" width="0.1524" layer="91"/>
@@
 </segment>
 </net>
-<net name="IO26" class="0">
+<net name="1IO26" class="0">
 <segment>
 <pinref part="IC201" gate="G$1" pin="I26"/>
@@
 </segment>
 </net>
-<net name="IO42" class="0">
+<net name="1IO42" class="0">
 <segment>
 <pinref part="IC201" gate="G$1" pin="I42"/>
@@
 <pinref part="IC201" gate="G$1" pin="I01"/>
 </segment>
-</net>
-<net name="IO18" class="0">
+<segment>
+<wire x1="83.82" y1="60.96" x2="78.74" y2="60.96" width="0.1524" layer="91"/>
+<label x="78.74" y="60.96" size="1.27" layer="95" font="vector" rot="R180" xref="yes"/>
+<pinref part="J208" gate="G$1" pin="9"/>
+</segment>
+</net>
+<net name="1IO18" class="0">
 <segment>
 <pinref part="IC201" gate="G$1" pin="I18"/>
@@
 </segment>
 </net>
-<net name="IO17" class="0">
+<net name="1IO17" class="0">
 <segment>
 <pinref part="IC201" gate="G$1" pin="I17"/>
@@
 </segment>
 </net>
-<net name="IO15" class="0">
+<net name="1IO15" class="0">
 <segment>
 <pinref part="IC201" gate="G$1" pin="I15"/>
@@
 <label x="10.16" y="25.4" size="1.27" layer="95" font="vector" rot="R270" xref="yes"/>
 </segment>
-</net>
-<net name="IO16" class="0">
-<segment>
-<pinref part="IC201" gate="G$1" pin="I16"/>
-<wire x1="12.7" y1="27.94" x2="12.7" y2="25.4" width="0.1524" layer="91"/>
-<label x="12.7" y="25.4" size="1.27" layer="95" font="vector" rot="R270" xref="yes"/>
+<segment>
+<wire x1="93.98" y1="63.5" x2="99.06" y2="63.5" width="0.1524" layer="91"/>
+<label x="99.06" y="63.5" size="1.27" layer="95" font="vector" xref="yes"/>
+<pinref part="J208" gate="G$1" pin="8"/>
 </segment>
 </net>
@@
 <pinref part="IC201" gate="G$1" pin="I00"/>
 </segment>
-</net>
-<net name="IO21" class="0">
+<segment>
+<label x="-43.18" y="48.26" size="1.27" layer="95" font="vector" xref="yes"/>
+<pinref part="J202" gate="G$1" pin="6"/>
+<wire x1="-48.26" y1="48.26" x2="-43.18" y2="48.26" width="0.1524" layer="91"/>
+</segment>
+<segment>
+<label x="99.06" y="71.12" size="1.27" layer="95" font="vector" xref="yes"/>
+<pinref part="J208" gate="G$1" pin="2"/>
+<wire x1="93.98" y1="71.12" x2="99.06" y2="71.12" width="0.1524" layer="91"/>
+</segment>
+</net>
+<net name="1IO21" class="0">
 <segment>
 <pinref part="IC201" gate="G$1" pin="I21"/>
@@
 <net name="1IO35" class="0">
 <segment>
-<label x="99.06" y="71.12" size="1.27" layer="95" font="vector" xref="yes"/>
-<pinref part="J208" gate="G$1" pin="2"/>
-<wire x1="93.98" y1="71.12" x2="99.06" y2="71.12" width="0.1524" layer="91"/>
-</segment>
-<segment>
 <wire x1="40.64" y1="43.18" x2="43.18" y2="43.18" width="0.1524" layer="91"/>
 <label x="43.18" y="43.18" size="1.27" layer="95" font="vector" xref="yes"/>
 <pinref part="IC201" gate="G$1" pin="I35"/>
 </segment>
-<segment>
-<label x="-43.18" y="48.26" size="1.27" layer="95" font="vector" xref="yes"/>
-<pinref part="J202" gate="G$1" pin="6"/>
-<wire x1="-48.26" y1="48.26" x2="-43.18" y2="48.26" width="0.1524" layer="91"/>
-</segment>
 </net>
 <net name="1IO2" class="0">
-<segment>
-<wire x1="93.98" y1="63.5" x2="99.06" y2="63.5" width="0.1524" layer="91"/>
-<label x="99.06" y="63.5" size="1.27" layer="95" font="vector" xref="yes"/>
-<pinref part="J208" gate="G$1" pin="8"/>
-</segment>
 <segment>
 <wire x1="0" y1="66.04" x2="-2.54" y2="66.04" width="0.1524" layer="91"/>
@@
 <pinref part="IC201" gate="G$1" pin="I02"/>
 </segment>
-</net>
-<net name="1IO46" class="0">
 <segment>
 <wire x1="93.98" y1="60.96" x2="99.06" y2="60.96" width="0.1524" layer="91"/>
@@
 <pinref part="J208" gate="G$1" pin="10"/>
 </segment>
+</net>
+<net name="1IO46" class="0">
 <segment>
 <wire x1="40.64" y1="71.12" x2="43.18" y2="71.12" width="0.1524" layer="91"/>
@@
 </net>
 <net name="1IO45" class="0">
-<segment>
-<wire x1="83.82" y1="60.96" x2="78.74" y2="60.96" width="0.1524" layer="91"/>
-<label x="78.74" y="60.96" size="1.27" layer="95" font="vector" rot="R180" xref="yes"/>
-<pinref part="J208" gate="G$1" pin="9"/>
-</segment>
 <segment>
 <wire x1="40.64" y1="68.58" x2="43.18" y2="68.58" width="0.1524" layer="91"/>
@@
 </segment>
 </net>
-<net name="I33" class="0">
+<net name="1IO33" class="0">
 <segment>
 <pinref part="IC201" gate="G$1" pin="I33"/>
@@
 </segment>
 </net>
+<net name="1IO16" class="0">
+<segment>
+<pinref part="IC201" gate="G$1" pin="I16"/>
+<wire x1="12.7" y1="27.94" x2="12.7" y2="25.4" width="0.1524" layer="91"/>
+<label x="12.7" y="25.4" size="1.27" layer="95" font="vector" rot="R270" xref="yes"/>
+</segment>
+</net>
