File: extras/esp32_hub75/eagle/esp32_hub75.brd (EAGLE design)
At the start: 99.8 x 53.1 mm, 64 parts, among them IC1 DS3231W, IC2 DC-DC-STEP-DOWN-LM2596, IC3 BH1750, IC4 1117 3V3, IC5 BME280, IC6 ESP32, IC7 74HCT245DW, IC8 74HCT245DW, J1 12V, J2 COM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

Commit message: upg board
Connections:
- net IO35: now also R9.2, X1.2; no longer R1.2, R2.2, R3.1
- net SVN: now also R1.2, R2.2, R3.1; no longer R9.2, X1.2
Routing:
- net SVN: track 93.3 -> 76.8 mm
- net IO35: track 79.5 -> 91.5 mm, vias 4 -> 2
- net IO13: track 46.6 -> 47.4 mm
