File: extras/esp32_hub75/eagle/esp32_hub75.sch (EAGLE design)
At the start: 64 parts, among them IC1 DS3231W, IC2 DC-DC-STEP-DOWN-LM2596, IC3 BH1750, IC4 1117 3V3, IC5 BME280, IC6 ESP32, IC7 74HCT245DW, IC8 74HCT245DW, J1 12V, J2 COM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

Commit message: upg board
Connections:
- net IO35: now also R9.2, X1-2.S; no longer R1.P$2, R2.2, R3.1
- net SVN: now also R1.P$2, R2.2, R3.1; no longer R9.2, X1-2.S
Other:
- moved on the sheet: C14, C15, C16, C17, C18, C3, C4, C6, D3, HA1, IC3, J3-1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
