File: extras/Main_board/eagle/clock10.brd (EAGLE design)
At the start: 91 x 96 mm, 120 parts, among them IC101 DC-DC-STEP-DOWN-LM2596, IC102 DS3231W, IC103 1117 3V3, IC104 ZOPT2201, IC105 BME280, IC106 74AC245DW, IC107 74AC245DW, IC201 ESP32S2, IC202 ESP12F, IC203 ESP32C3-MODULE13U, IC204 ESP12F, IC301 1117 3V3, IC302 BME280, J101 12V, J102 IN, J104 4P-2.0, J105 4P-2.0, J201 USB_1, J202 COM, J203 COM, J204 COM, J205 COM, J206 USB_2, J207 OUT_2, J208 OUT_1, J209 OUT_3, J301 IN, SW101 PRG, SW102 RST, U101 SI7021, U301 SI7021, X101 +5V, X102 SHT22, X103 AM2320, X301 +5V, X302 DHT22, X303 AM2320

Commit message: add new boards
Parts:
- removed B101: SR2032, radiva5:CR2032
- removed C102, C202, C208, C209, C302, C303, C304, C306, C307: 0.1u, radiva5:0603-CAP
- removed C201, C203, C204: 10u, radiva5:0603-CAP
- removed C301: 100x5v, radiva5:CPOL-RADIAL-100UF-25V
- removed C305: 100x3V, radiva5:CPOL-RADIAL-100UF-25V
- removed D201, D202, D203: IN5819, radiva5:SOD123
- removed IC201: ESP32S2, radiva5:ESP-12K
- removed IC202: ESP12F, esp8266modules:ESP12-SMD
- removed IC203: ESP32C3-MODULE13U, radiva5:ESP32C3-13U
- removed IC301: 1117 3V3, radiva5:SOT223
- removed IC302: BME280, radiva5:LGA-8-2.5X2.5
- removed J201: USB_1, radiva5:USB-B-MICRO-SMD_MY
- removed J202, J203, J204: COM, radiva5:2X03_SMT
- removed J206: USB_2, radiva5:USB-B-MICRO-SMD_MY
- removed J207: OUT_2, radiva5:2X8
- removed J208: OUT_1, radiva5:2X13
- removed J209: OUT_3, radiva5:2X8
- removed J301: IN, radiva5:2X04
- removed R101: 220k, radiva5:R0603
- removed R102: 100k, radiva5:R0603
- removed R103: 10K, radiva5:SNR2-3.0
- removed R201, R202, R203, R204, R205, R302, R303: 10k, radiva5:R0603
- removed R301: 1k, radiva5:R0603
- removed SJ201, SJ202: L/W, radiva5:MICROBUILDER_SOLDERJUMPER_ARROW_NOPASTE_3
- removed SJ203: DHT, radiva5:MICROBUILDER_SOLDERJUMPER_ARROW_NOPASTE
- removed SJ301: i2c_pullup, radiva5:MICROBUILDER_SOLDERJUMPER_ARROW_NOPASTE
- removed U101, U301: SI7021, radiva5:DFN-6-3X3-SI7021
- removed X101, X301: +5V, con-molex:70543-02
- removed X102: SHT22, con-molex:70543-04
- removed X103, X303: AM2320, con-molex:70543-04
- removed X302: DHT22, con-molex:70543-04
- added C1: 0.1u, radiva5:0603-CAP
- added G103: CH291-1220LF09, clock02:CH23-09LF
- added IC108: 74AC245DW, 74xx-eu:SO20W
- added J1: FR, radiva5:1X03
- added J107: (no value), radiva5:2X05_IDC
- added J108, J109: 4P-2.0, radiva5:HW4-2.0
- added R210, R211: 2k, radiva5:R0603
- added R3, R4: 47k, radiva5:R0603
- added SJ1: PR POS/NEG, radiva5:MICROBUILDER_SOLDERJUMPER_ARROW_NOPASTE_3
- G101: value CH291-1220LF -> SR2032; device clock02:CH291-1220LF -> radiva5:CR2032
- G102: value CH291-1220LF09 -> CH291-1220LF; device clock02:CH23-09LF -> clock02:CH291-1220LF
- IC105: value BME280 -> SI7021; device radiva5:LGA-8-2.5X2.5 -> radiva5:DFN-6-3X3-SI7021
- IC106: value 74AC245DW -> BME280; device 74xx-eu:SO20W -> radiva5:LGA-8-2.5X2.5
- J102: value IN -> +5V; device radiva5:2X13 -> con-molex:70543-02
- J103: value (none) -> SHT22; device radiva5:2X05_IDC -> con-molex:70543-04
- J104: value 4P-2.0 -> IN; device radiva5:HW4-2.0 -> radiva5:2X13
- J105: value 4P-2.0 -> AM2320; device radiva5:HW4-2.0 -> con-molex:70543-04
- R207, R208: value 2k -> 10k
- moved IC106 54.3 mm to (42.7, -12.7), flipped to the top
- moved J104 39.1 mm to (3.05, 26.4)
- moved R206 32.5 mm to (-1.78, -25.1), turned to 0 degrees
- moved J102 31.9 mm to (28.4, 45.7), turned to 180 degrees
- moved R207 19.3 mm to (-1.78, -42.7)
- moved IC107 17.0 mm to (20.3, 36.8)
- moved J105 17.0 mm to (48.0, -13.2), turned to 270 degrees
- moved J103 16.1 mm to (25.4, 5.59), turned to 90 degrees
- moved R208 8.87 mm to (-1.78, -31.5), turned to 0 degrees
- moved G102 7.37 mm to (9.40, -11.3), turned to 0 degrees
- moved G101 5.72 mm to (9.40, -5.59), turned to 270 degrees
- moved IC105 5.09 mm to (42.4, -7.62), turned to 0 degrees
- moved LED101 0.25 mm to (0.76, -17.0), turned to 90 degrees
- renumbered C205 to C213, C206 to C214, C207 to C215, IC204 to IC206, J205 to J213, JP101 to J106, R209 to R212
Connections:
- net 4IO12 renamed 6IO12
- net 4IO13 renamed 6IO13
- net 4IO14 renamed 6IO14
- net 4IO15 renamed 6IO15
- net 4IO16 renamed 6IO16
- net 4IO4 renamed 6IO4
- net 4IO5 renamed 6IO5
- net 4RX0 renamed 6RX0
- net 4TX0 renamed 6TX0
- removed net +3V3_1: C201.2, C202.2, D203.C, IC201.VCC, J208.4
- removed net +3V3_2: C204.2, C209.2, D202.C, IC203.3V3, J207.4
- removed net +3V3_3: C203.2, C208.2, D201.C, IC202.VCC, J209.4, R201.2
- removed net +3V3_4: C214.2, C215.2, IC206.VCC, J213.6, LED201.A, LED202.A, R203.2, R205.2
- removed net +3V3_S: C303.2, C304.1, C305.1, C306.2, C307.2, IC301.2, IC301.4, IC302.6, IC302.8, J301.1, R301.1, SJ301.1, U301.VDD, X302.1, X303.1
- removed net +5V_1: J201.VBUS, J208.6
- removed net +5V_2: J206.VBUS, J207.6
- removed net +5V_3: J209.6
- removed net +5V_S: C301.1, C302.1, IC301.3, J301.3, X301.2
- removed net 1EN: IC201.RST, J202.1, J208.1
- removed net 1I037: IC201.I37, J208.11
- removed net 1IO0: IC201.I00, J202.6, J208.2
- removed net 1IO1: IC201.I01, J208.9
- removed net 1IO10: IC201.I10, J208.22
- removed net 1IO11: IC201.I11, J208.23
- removed net 1IO12: IC201.I12, J208.24
- removed net 1IO13: IC201.I13, J208.20
- removed net 1IO14: IC201.I14, J208.21
- removed net 1IO15: IC201.I15, J208.8
- removed net 1IO16: IC201.I16
- removed net 1IO17: IC201.I17
- removed net 1IO18: IC201.I18
- removed net 1IO19: IC201.I19, J201.D-
- removed net 1IO2: IC201.I02, J208.10
- removed net 1IO20: IC201.I20, J201.D+
- removed net 1IO21: IC201.I21
- removed net 1IO26: IC201.I26
- removed net 1IO3: IC201.I03, J208.5
- removed net 1IO33: IC201.I33
- removed net 1IO34: IC201.I34, J208.12
- removed net 1IO35: IC201.I35
- removed net 1IO36: IC201.I36, J208.19
- removed net 1IO38: IC201.I38
- removed net 1IO39: IC201.I39, J208.14
- removed net 1IO4: IC201.I04, J208.7
- removed net 1IO40: IC201.I40, J208.15
- removed net 1IO41: IC201.I41, J208.16
- removed net 1IO42: IC201.I42
- removed net 1IO45: IC201.I45
- removed net 1IO46: IC201.I46
- removed net 1IO5: IC201.I05, J208.26
- removed net 1IO6: IC201.I06, J208.18
- removed net 1IO7: IC201.I07, J208.17
- removed net 1IO8: IC201.I08, J208.13
- removed net 1IO9: IC201.I09, J208.25
- removed net 1RX0: IC201.RX, J202.5
- removed net 1TX0: IC201.TX, J202.3
- removed net 2D+: IC203.IO19, J206.D+
- removed net 2D-: IC203.IO18, J206.D-
- removed net 2EN: IC203.EN, J204.1, J207.1
- removed net 2IO0: IC203.IO0, J207.8
- removed net 2IO1: IC203.IO1, J207.7
- removed net 2IO10: IC203.IO10, J207.15
- removed net 2IO2: IC203.IO2, J207.5
- removed net 2IO3: IC203.IO3, J207.12
- removed net 2IO4: IC203.IO4, SJ201.1
- removed net 2IO5: IC203.IO5, J207.9
- removed net 2IO6: IC203.IO6, J207.10
- removed net 2IO7: IC203.IO7, J207.16
- removed net 2IO8: IC203.IO8, J207.14
- removed net 2IO9: IC203.IO9, J204.6, J207.2
- removed net 2RX0: IC203.RX0, J204.5
- removed net 2TX0: IC203.TX0, J204.3
- removed net 3ADC: IC202.ADC, J209.7, R202.1
- removed net 3EN: IC202.RESET, J203.1, J209.1
- removed net 3IO0: IC202.GPIO0, J203.6, J209.2
- removed net 3IO12: IC202.GPIO12, J209.5
- removed net 3IO13: IC202.GPIO13, J209.16
- removed net 3IO14: IC202.GPIO14, J209.15
- removed net 3IO15: IC202.GPIO15, J209.12, R206.2
- removed net 3IO16: IC202.GPIO16, J209.14
- removed net 3IO2: IC202.GPIO2, SJ202.1, SJ203.2
- removed net 3IO4: IC202.GPIO4, J209.9
- removed net 3IO5: IC202.GPIO5, J209.10
- removed net 3RX0: IC202.RXD0, J203.5
- removed net 3TX0: IC202.TXD0, J203.3
- removed net 4EN: C213.2, IC206.RESET, R203.1
- removed net 4IO0: IC206.GPIO0, R208.1
- removed net 4IO2: IC206.GPIO2, R207.1
- removed net COM_VCC2: D201.A, J203.2
- removed net I2C_SCL_S: IC302.4, J301.7, R302.2, U301.SCK, X303.4
- removed net I2C_SDA_S: IC302.3, J301.8, R303.2, U301.DATA, X303.2
- removed net IN2_A: J207.13, SJ201.2
- removed net IN3_DHT: J209.8, SJ203.1
- removed net IN_DHT_S: J301.5, R301.2, X302.2
- removed net N$13: J209.13, SJ202.2
- removed net N$14: J209.11, SJ202.3
- removed net N$15: J207.11, SJ201.3
- removed net N$3: R302.1, R303.1, SJ301.2
- removed net N$6: IC202.CH_PD, R201.1
- new net +3V3_6: C214.2, C215.2, IC206.VCC, J213.6, LED201.A, LED202.A, R206.2, R208.2
- new net 6EN: C213.2, IC206.RESET, R206.1
- new net 6IO0: IC206.GPIO0, R210.1
- new net 6IO2: IC206.GPIO2, R211.1
- net +3V3: now also C1.1, IC105.VDD, IC106.6, IC106.8, J103.1, J105.1, J108.3, J109.3, R3.2; no longer C102.1, IC105.6, IC105.8, J102.3, J105.3, R101.2, U101.VDD, X102.1, X103.1
- net +5V: now also J102.2, J104.5; no longer J102.5, X101.2
- net A(CS_CLK): now also IC108.18, J107.8; no longer IC107.18, J103.8
- net B(CS): now also IC108.17, J107.7; no longer IC107.17, J103.7
- net BLUE1: now also IC107.16; no longer IC106.16
- net BLUE2: now also IC107.13; no longer IC106.13
- net BUZZER: now also IC108.11; no longer IC107.11
- net C(LOCK): now also IC108.16, J107.10; no longer IC107.16, J103.10
- net CLOCK: now also IC107.12; no longer IC106.12
- net D(ATA): now also IC108.15, J107.9; no longer IC107.15, J103.9
- net E: now also IC108.14; no longer IC107.14
- net GND: now also C1.2, G102.-, G103.P"-", IC105.GND, IC106.1, IC106.7, IC108.10, IC108.19, J102.1, J105.3, J107.3, J107.4, J107.5, J107.6, J108.4, J109.4, R207.2, R4.1; no longer B101.-, C102.2, C201.1, C202.1, C203.1, C204.1, C208.1, C209.1, C301.2, C302.2, C303.1, C304.2, C305.2, C306.1, C307.1, G102.P"-", IC105.1, IC105.7, IC106.10, IC106.19, IC201.GND1, IC201.GND2, IC201.GND3, IC201.PAD0, IC201.PAD1, IC201.PAD2, IC201.PAD3, IC201.PAD4, IC201.PAD5, IC201.PAD6, IC201.PAD7, IC201.PAD8, IC202.GND, IC203.GND, IC301.1, IC302.1, IC302.7, J102.4, J103.3, J103.5, J103.6, J105.4, J201.GND, J201.SH@1, J201.SH@2, J201.SH@3, J201.SH@4, J201.SH@5, J201.SH@6, J202.4, J203.4, J204.4, J206.GND, J206.SH@1, J206.SH@2, J206.SH@3, J206.SH@4, J206.SH@5, J206.SH@6, J207.3, J208.3, J209.3, J301.2, R102.1, R103.1, R202.2, R204.2, R206.1, U101.GND, U301.GND, X101.1, X102.4, X103.3, X301.1, X302.4, X303.3
- net GREEN1: now also IC107.17; no longer IC106.17
- net GREEN2: now also IC107.14; no longer IC106.14
- net I2C_SCL: now also IC105.SCK, IC106.4, J104.9, J105.4, J108.1, J109.1; no longer IC105.4, J102.9, J104.1, J105.1, U101.SCK, X103.4
- net I2C_SDA: now also IC105.DATA, IC106.3, J104.10, J108.2, J109.2; no longer IC105.3, J102.10, J104.2, U101.DATA, X103.2
- net IN_A: now also IC108.2, J104.14; no longer IC107.2, J102.14
- net IN_B: now also IC108.3, J104.13; no longer IC107.3, J102.13
- net IN_BLUE1: now also IC107.4, J104.22; no longer IC106.4, J102.22
- net IN_BLUE2: now also IC107.7, J104.23; no longer IC106.7, J102.23
- net IN_BUZZER: now also IC108.9, J104.11; no longer IC107.9, J102.11
- net IN_C: now also IC108.4, J104.16; no longer IC107.4, J102.16
- net IN_CLOCK: now also IC107.8, J104.26; no longer IC106.8, J102.26
- net IN_D: now also IC108.5, J104.15; no longer IC107.5, J102.15
- net IN_DHT: now also J103.2, J104.7; no longer J102.7, X102.2
- net IN_E: now also IC108.6, J104.18; no longer IC107.6, J102.18
- net IN_GREEN1: now also IC107.3, J104.19; no longer IC106.3, J102.19
- net IN_GREEN2: now also IC107.6, J104.24; no longer IC106.6, J102.24
- net IN_LATCH: now also IC107.9, J104.25; no longer IC106.9, J102.25
- net IN_LED: now also IC108.8, J104.12; no longer IC107.8, J102.12
- net IN_OE: now also IC108.7, J104.17; no longer IC107.7, J102.17
- net IN_RED1: now also IC107.2, J104.20; no longer IC106.2, J102.20
- net IN_RED2: now also IC107.5, J104.21; no longer IC106.5, J102.21
- net LATCH: now also IC107.11; no longer IC106.11
- net LED: now also IC108.12; no longer IC107.12
- net N$10: now also R207.1; no longer R204.1
- net N$11: now also R210.2; no longer R208.2
- net N$12: now also R211.2; no longer R207.2
- net N$4: now also J1.3, R3.1, SJ1.3; no longer D203.A, J202.2
- net N$52: now also G102.+, G103.P1"+"; no longer B101.+, G102.P1"+"
- net N$8: now also J1.1, R4.2, SJ1.2; no longer D202.A, J204.2
- net N$9: now also R208.1; no longer R205.1
- net OE: now also IC108.13; no longer IC107.13
- net PHOTO_RES: now also J1.2, J104.8, SJ1.1; no longer J102.8, R101.1, R102.2, R103.2
- net PRG_BTN: now also J104.1; no longer J102.1
- net RED1: now also IC107.18; no longer IC106.18
- net RED2: now also IC107.15; no longer IC106.15
- net RST_BTN: now also J104.2; no longer J102.2
- net SQW: now also J104.6; no longer J102.6
- net VCC: now also IC108.1, IC108.20; no longer IC106.1, IC106.20
- net V_SPI: now also J107.1, J107.2; no longer J103.1, J103.2
Routing:
- net +3V3_S: track 70.7 -> 0.00 mm, vias 3 -> 0
- net +3V3_1: track 58.7 -> 0.00 mm, vias 1 -> 0
- net +5V_1: track 53.5 -> 0.00 mm, vias 1 -> 0
- net 1EN: track 52.4 -> 0.00 mm, vias 1 -> 0
- net 1IO0: track 44.2 -> 0.00 mm, vias 1 -> 0
- net 1IO3: track 40.2 -> 0.00 mm, vias 2 -> 0
- net 2EN: track 39.8 -> 0.00 mm, vias 1 -> 0
- net I2C_SDA_S: track 39.4 -> 0.00 mm, vias 2 -> 0
- net 3EN: track 39.1 -> 0.00 mm, vias 2 -> 0
- net 1IO1: track 37.8 -> 0.00 mm, vias 3 -> 0
- net 1IO4: track 37.6 -> 0.00 mm, vias 2 -> 0
- net +5V_S: track 37.1 -> 0.00 mm
- net 1IO2: track 36.6 -> 0.00 mm, vias 3 -> 0
- net +3V3_2: track 36.2 -> 0.00 mm, vias 1 -> 0
- net +3V3_3: track 33.0 -> 0.00 mm, vias 2 -> 0
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Other:
- board size 91 x 96 mm -> 57.1 x 96.3 mm
- board text removed: "00 3V 5V DH 05 15 16 13"
- board text removed: "07 08 03 06 00 5V 3V 09"
- board text removed: "10 _A 15 05 01 02 GD EN"
- board text removed: "35 3V 5V 02 46 34 39 41 06 13 10 12 05"
- board text removed: "EN GD 03 04 45 37 08 40 07 36 14 11 09"
- board text removed: "EN GD 12 AD 04 LD _A 14"
- board text removed: "EN GD SQ FR SD LD _A _C"
- board text removed: "PG 3V 5V DH SC SN _B _D"
- board text removed: "SC"
- board text removed: "SD"
- board text removed: "_C _A LD SD FR SQ GD EN"
- board text removed: "_D _B SN SC DH 5V 3V PG"

Commit message: bug fix
Parts:
- moved IC104 45.0 mm to (-8.26, -12.2)
- moved IC206 45.0 mm to (-37.1, -39.1)
- moved J213 45.0 mm to (-37.1, -36.8)
- moved LED102 45.0 mm to (2.79, -3.56)
- moved C1 45.0 mm to (-24.4, -17.8)
- moved C101 45.0 mm to (-11.2, -9.02)
- moved C103 45.0 mm to (0.51, -16.0)
- moved C104 45.0 mm to (-9.40, -6.10)
- moved C105 45.0 mm to (-9.14, -3.81)
- moved C106 45.0 mm to (0.51, -10.9)
- moved C107 45.0 mm to (-18.9, -1.27)
- moved C108 45.0 mm to (-17.8, -6.35)
- moved C109 45.0 mm to (-5.71, -12.4)
- moved C110 45.0 mm to (-13.6, -13.2)
- moved C111 45.0 mm to (-1.52, -10.9)
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Routing:
- net +3V3_S: track 0.00 -> 147.3 mm, vias 0 -> 5
- net N$6: track 0.00 -> 100.0 mm
- net N$13: track 0.00 -> 100.0 mm
- net +3V3_3: track 0.00 -> 83.5 mm
- net +3V3_4: track 0.00 -> 81.6 mm
- net +5V_S: track 0.00 -> 76.6 mm, vias 0 -> 6
- net +3V3_2: track 0.00 -> 68.3 mm
- net I2C_SDA_S: track 0.00 -> 61.0 mm, vias 0 -> 4
- net I2C_SCL_S: track 0.00 -> 60.8 mm, vias 0 -> 2
- net 4EN: track 0.00 -> 59.3 mm
- net 3EN: track 0.00 -> 59.3 mm
- net 4IO21: track 0.00 -> 53.9 mm
- net 3IO0: track 0.00 -> 45.7 mm
- net 3IO4: track 0.00 -> 45.5 mm
- net 2EN: track 0.00 -> 44.0 mm
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- added copper zone on layer 1, net GND1
- added copper zone on layer 16, net GND1
- added copper zone on layer 1, net RET1
- added copper zone on layer 16, net RET1
