File: extras/Main_board/eagle/clock10.sch (EAGLE design)
At the start: 77 parts, among them IC101 DC-DC-STEP-DOWN-LM2596, IC102 DS3231W, IC103 1117 3V3, IC104 ZOPT2201, IC105 SI7021, IC106 BME280, IC107 74AC245DW, IC108 74AC245DW, IC206 ESP12F, J1 FR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

Commit message: add m7219 test
Changed lines of the file:
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@@
 <segment>
 <wire x1="93.98" y1="137.16" x2="91.44" y2="137.16" width="0.1524" layer="91"/>
-<label x="83.312" y="139.7" size="1.27" layer="95" rot="R180"/>
+<label x="78.74" y="137.16" size="1.27" layer="95" font="vector" rot="R180" xref="yes"/>
 <pinref part="SW101" gate="G$1" pin="B"/>
 <pinref part="R109" gate="G$1" pin="1"/>
-<wire x1="91.44" y1="137.16" x2="73.66" y2="137.16" width="0.1524" layer="91"/>
+<wire x1="91.44" y1="137.16" x2="78.74" y2="137.16" width="0.1524" layer="91"/>
 <wire x1="88.9" y1="142.24" x2="91.44" y2="142.24" width="0.1524" layer="91"/>
 <wire x1="91.44" y1="142.24" x2="91.44" y2="137.16" width="0.1524" layer="91"/>
