File: extras/clock_13/clock14.sch (EAGLE design)
At the start: 74 parts, among them IC1 VS1838, IC102 ESP32, IC103 ESP32C3-MODULE13U, IC3 IRM-H638T, J101 COM, J102 COM, J107 COM, J2 4P-2.0, K101 SRD-05VDC SL-C, K102 SRD-05VDC SL-C, SW1 PRG, SW101 RST, SW102 PRG, SW103 RST, SW104 RST, SW105 PRG, SW106 PRG, T101 S8050, T102 S8050, U101 AP2112, U102 AP2112, U103 AP2112, X1 SHT22

Commit message: add m7219 test
Connections:
- net 4IO21: now also J112.9; no longer J112.24
- net 4IO23: now also J112.24; no longer J112.9

Commit message: 1111
Parts:
- removed C104: 500u, radiva5:CAP_POLPTH1
- removed IC102: ESP32, radiva5:ESP32-MODULEDUAL
- removed IC103: ESP32C3-MODULE13U, radiva5:ESP32C3-MODULE13U
- removed J102: COM, radiva5:HEADER-2X3SMT
- removed J109: (no value), radiva5:USB_MICRO-BFEMALE_SMT_
- removed J111: (no value), radiva5:HEADER-2X8
- removed R102, R109, R112: 10k, radiva5:R-EU_R0603
- removed R104: 100k, radiva5:R-EU_R0603
- removed R107: (no value), radiva5:R-EU_R0603
- removed SW104: RST, radiva5:MICROSWITCH-BUTTON
- added C17: 4.7u, radiva5:CAP0603-CAP
- added IC4: VS1838, radiva5:VS1838
- added IC5: IRM-H638T, radiva5:IRM-H638T
- added J11: (no value), radiva5:CONN_02
- added J14: (no value), radiva5:HEADER-2X8
- added J16: 4P-2.0, radiva5:GROVE-CONNECTOR-DIP(4P-2.0)
- added R12, R17, R5: 10k, radiva5:R-EU_R0603
- added R14: PHOTORESISTOR-5528-10K, radiva5:PHOTORESISTOR-5528-10K(2P-5.0X4.2MM)
- added R16: 100, radiva5:R-EU_R0603
- added SW7: PRG, radiva5:MICROSWITCH-BUTTON
- C2: value 4.7u -> 500u; device radiva5:CAP0603-CAP -> radiva5:CAP_POLPTH1
- IC1: value VS1838 -> ESP32C3-MODULE13U; device radiva5:VS1838 -> radiva5:ESP32C3-MODULE13U
- IC2: value (none) -> ESP8266
- IC3: value IRM-H638T -> ESP32; device radiva5:IRM-H638T -> radiva5:ESP32-MODULEDUAL
- J1: value (none) -> COM; device radiva5:HEADER-2X8 -> radiva5:HEADER-2X3SMT
- J2: value 4P-2.0 -> (none); device radiva5:GROVE-CONNECTOR-DIP(4P-2.0) -> radiva5:HEADER-2X8
- J3: device radiva5:CONN_02 -> radiva5:USB_MICRO-BFEMALE_SMT_
- R1: value PHOTORESISTOR-5528-10K -> 10k; device radiva5:PHOTORESISTOR-5528-10K(2P-5.0X4.2MM) -> radiva5:R-EU_R0603
- R11: value 100 -> (none)
- R2: value 10k -> 100k
- SW1: value PRG -> RST
- renumbered C101 to C7, C102 to C6, C103 to C11, C105 to C3, C106 to C14, C107 to C12, C108 to C15, C109 to C8, C110 to C4, C111 to C10, C112 to C16, C113 to C5, C114 to C13, C115 to C9, C116 to C1, D101 to D2, D102 to D1, IC101 to IC2, J101 to J6, J103 to J13, J104 to J12, J105 to J10, J106 to J9, J107 to J7, J108 to J5, J112 to J8, J113 to J4, K101 to K2, K102 to K1, R101 to R4, R103 to R8, R105 to R7, R106 to R15, R108 to R13, R110 to R9, R111 to R6, SJ101 to SJ1, SJ102 to SJ3, SJ103 to SJ2, SW101 to SW5, SW102 to SW6, SW103 to SW3, SW105 to SW4, SW106 to SW2, T101 to T2, T102 to T1, U101 to U2, U102 to U1, U103 to U3, X1 to J15
Connections:
- net +3V3_1: now also IC4.VCC, J14.4, J16.3, R12.1, R16.2, R17.1; no longer IC1.VCC, J1.4, J2.3, R10.1, R11.2, R2.1
- net +3V3_2: now also C2.+, IC1.VCC, J1.2, J2.4, R1.2; no longer C104.+, IC103.VCC, J102.2, J111.4, R112.2
- net +3V3_3: now also R5.1; no longer R3.1
- net +3V3_4: now also IC3.3V3; no longer IC102.3V3
- net +5V_1: now also J11.2, J14.6; no longer J1.6, J3.2
- net +5V_2: now also J2.6, J3.VBUS, R2.1; no longer J109.VBUS, J111.6, R104.1
- net 1ADC: now also J14.7, R14.P$1; no longer J1.7, R1.P$1
- net 1EN: now also J14.1; no longer J1.1
- net 1IO0: now also J14.2; no longer J1.2
- net 1IO12: now also IC4.OUT, IC5.OUT, J14.5, R17.2; no longer IC1.OUT, IC3.OUT, J1.5, R10.2
- net 1IO13: now also J14.16; no longer J1.16
- net 1IO14: now also J14.15, R10.2; no longer J1.15, R109.2
- net 1IO15: now also J14.12; no longer J1.12
- net 1IO16: now also J14.14; no longer J1.14
- net 1IO2: now also J14.8, SW7.B; no longer J1.8, SW1.B
- net 1IO4: now also J14.9, J16.2; no longer J1.9, J2.2
- net 1IO5: now also J14.10, J16.1; no longer J1.10, J2.1
- net 2D+: now also IC1.IO19, J3.D+; no longer IC103.IO19, J109.D+
- net 2D-: now also IC1.IO18, J3.D-; no longer IC103.IO18, J109.D-
- net 2EN: now also IC1.EN, J1.1, J2.1, R1.1, SW1.B; no longer IC103.EN, J102.1, J111.1, R112.1, SW104.B
- net 2EN_P: now also R2.2; no longer R104.2
- net 2IO0: now also IC1.IO0, J2.8; no longer IC103.IO0, J111.8
- net 2IO1: now also IC1.IO1, J2.7; no longer IC103.IO1, J111.7
- net 2IO10: now also IC1.IO10, J2.15; no longer IC103.IO10, J111.15
- net 2IO2: now also IC1.IO2, J2.5; no longer IC103.IO2, J111.5
- net 2IO3: now also IC1.IO3, J2.12; no longer IC103.IO3, J111.12
- net 2IO4: now also IC1.IO4; no longer IC103.IO4
- net 2IO5: now also IC1.IO5, J2.9; no longer IC103.IO5, J111.9
- net 2IO6: now also IC1.IO6, J2.10; no longer IC103.IO6, J111.10
- net 2IO7: now also IC1.IO7, J2.16; no longer IC103.IO7, J111.16
- net 2IO8: now also IC1.IO8, J2.14; no longer IC103.IO8, J111.14
- net 2IO9: now also IC1.IO9, J1.6, J2.2; no longer IC103.IO9, J102.6, J111.2
- net 2RX0: now also IC1.RX0, J1.5; no longer IC103.RX0, J102.5
- net 2TX0: now also IC1.TX0, J1.3; no longer IC103.TX0, J102.3
- net 3ADC: now also R3.1; no longer R102.1
- net 3IO2: now also R5.2; no longer R3.2
- net 4EN: now also IC3.EN; no longer IC102.EN
- net 4IO0: now also IC3.IO0; no longer IC102.IO0
- net 4IO12: now also IC3.IO12; no longer IC102.IO12
- net 4IO13: now also IC3.IO13; no longer IC102.IO13
- net 4IO14: now also IC3.IO14; no longer IC102.IO14
- net 4IO15: now also IC3.IO15; no longer IC102.IO15
- net 4IO16: now also IC3.I16; no longer IC102.I16
- net 4IO17: now also IC3.I17; no longer IC102.I17
- net 4IO18: now also IC3.IO18; no longer IC102.IO18
- net 4IO19: now also IC3.IO19; no longer IC102.IO19
- net 4IO2: now also IC3.IO2; no longer IC102.IO2
- net 4IO21: now also IC3.IO21; no longer IC102.IO21
- net 4IO22: now also IC3.IO22; no longer IC102.IO22
- net 4IO23: now also IC3.IO23; no longer IC102.IO23
- net 4IO25: now also IC3.IO25; no longer IC102.IO25
- net 4IO26: now also IC3.IO26; no longer IC102.IO26
- net 4IO27: now also IC3.IO27; no longer IC102.IO27
- net 4IO32: now also IC3.IO32; no longer IC102.IO32
- net 4IO33: now also IC3.IO33; no longer IC102.IO33
- net 4IO34: now also IC3.IO34; no longer IC102.IO34
- net 4IO35: now also IC3.IO35; no longer IC102.IO35
- net 4IO4: now also IC3.IO4; no longer IC102.IO4
- net 4IO5: now also IC3.IO5; no longer IC102.IO5
- net 4RX0: now also IC3.RXD0; no longer IC102.RXD0
- net 4SVN: now also IC3.SENSOR_VN; no longer IC102.SENSOR_VN
- net 4SVP: now also IC3.SENSOR_VP; no longer IC102.SENSOR_VP
- net 4TX0: now also IC3.TXD0; no longer IC102.TXD0
- net GND: now also C17.2, C2.-, IC3.GND@1, IC3.GND@15, IC3.GND@38, IC3.GND@39, IC4.GND, IC5.GND, IC5.GND1, J1.4, J11.1, J14.3, J16.4, J2.3, J3.GND, J3.SHIELD, R11.1, R3.2, SW7.A, SW7.SH; no longer C104.-, C2.2, IC102.GND@1, IC102.GND@15, IC102.GND@38, IC102.GND@39, IC103.GND, IC3.GND, IC3.GND1, J1.3, J102.4, J109.GND, J109.SHIELD, J111.3, J2.4, J3.1, R102.2, R107.1, SW104.A, SW104.SH
- net IN2_A: now also J2.13; no longer J111.13
- net IN2_LED: now also J2.11; no longer J111.11
- net N$10: now also R12.2, R14.P$2; no longer R1.P$2, R2.2
- net N$15: now also C17.1, IC5.VCC, R16.1; no longer C2.1, IC3.VCC, R11.1
- net N$3: now also R10.1, R11.2; no longer R107.2, R109.1
Other:
- moved on the sheet: R10, R11, R2, R3, SW1
